File: elec/layout/default/drv5053raqdbzr.kicad_pcb (KiCad board)
At the start: 2 copper layers, 225.7 x 100.8 mm, 0 parts

Commit message: initial design
Parts:
- added C1: 16V 100nF X7R ±10% 0402 Multilayer Ceramic Capacitors MLCC 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, lib:C0402, F.Cu at (160.3, 93.7)
- added C2: 16V 100nF X7R ±10% 0402 Multilayer Ceramic Capacitors MLCC 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, lib:C0402, F.Cu at (160.3, 90.4)
- added R1: 62.5mW Thick Film Resistors ±100ppm/℃ ±1% 3.24kΩ 0402 Chip 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, lib:R0402, F.Cu at (162.1, 89.8)
- added U1: , lib:SOT-23-3_L2.9-W1.3-P0.95-LS2.4-BR, F.Cu at (161.8, 92.1)
Routing:
- net vcc: track 0.00 -> 2.92 mm
- net gnd: track 0.00 -> 2.68 mm
- net ic-vcc: track 0.00 -> 1.36 mm
- net vcc-1: track 0.00 -> 1.26 mm
